File: hardware/strip/strip-cover/strip-cover.kicad_pcb (KiCad board)
At the start: 2 copper layers, 66 x 18 mm, 7 parts

Commit message: Replace Order_Number
Parts:
- H1: value MountingHole_1mm -> 1mm
- H2, H3: value Mounting_Hole -> 2mm_Pad_5.2mm
- INFO1: value ORDER-NUMBER -> ~; footprint V2_Production:Order_Number -> V2_Production:Revision
- moved INFO1 2.25 mm to (150.0, 113.5)
