File: hardware/strip/strip.kicad_sch (KiCad schematic)
At the start: 36 parts, among them J101 Cortex, J102 DX07S016JA3, SW101 SKSG, SW102 SKSG, U101 ATSAMD51G, U102 TPS78433QWDRBRQ1, Y101 32k768

Commit message: Good Bye Imperial
Parts:
- C101, C102: footprint V2_Capacitor_SMD:C_0603 -> V2_Capacitor_SMD:C_1608; symbol V2_Capacitor:0603_18p -> V2_Capacitor:1608_18p
- C103: footprint V2_Capacitor_SMD:C_0603 -> V2_Capacitor_SMD:C_1608; symbol V2_Capacitor:0603_10u -> V2_Capacitor:1608_10u
- C104, C105, C106, C107: footprint V2_Capacitor_SMD:C_0603 -> V2_Capacitor_SMD:C_1608; symbol V2_Capacitor:0603_0u1 -> V2_Capacitor:1608_0u1
- C108, C109: footprint V2_Capacitor_SMD:C_0805 -> V2_Capacitor_SMD:C_2012; symbol V2_Capacitor:0805_10u -> V2_Capacitor:2012_10u
- D101: symbol V2_LED:0603_Orange -> V2_LED:1608_Orange
- R101: footprint V2_Resistor_SMD:R_0603 -> V2_Resistor_SMD:R_1608; symbol V2_Resistor:0603_100k -> V2_Resistor:1608_100k
- R102: footprint V2_Resistor_SMD:R_0603 -> V2_Resistor_SMD:R_1608; symbol V2_Resistor:0603_330R -> V2_Resistor:1608_330R
- R103, R104: footprint V2_Resistor_SMD:R_0603 -> V2_Resistor_SMD:R_1608; symbol V2_Resistor:0603_5k1 -> V2_Resistor:1608_5k1
Changed lines of the file:
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@@
 	)
 	(symbol
-		(lib_id "V2_Resistor:0603_5k1")
+		(lib_id "V2_Resistor:1608_5k1")
 		(at 212.09 93.98 90)
 		(unit 1)
@@
 			)
 		)
-		(property "Footprint" "V2_Resistor_SMD:R_0603"
+		(property "Footprint" "V2_Resistor_SMD:R_1608"
 			(at 227.838 93.98 0)
 			(hide yes)
@@
 	)
 	(symbol
-		(lib_id "V2_Capacitor:0603_0u1")
+		(lib_id "V2_Capacitor:1608_0u1")
 		(at 115.57 25.4 0)
 		(unit 1)
@@
 			)
 		)
-		(property "Footprint" "V2_Capacitor_SMD:C_0603"
+		(property "Footprint" "V2_Capacitor_SMD:C_1608"
 			(at 115.57 42.418 0)
 			(hide yes)
@@
 	)
 	(symbol
-		(lib_id "V2_LED:0603_Orange")
+		(lib_id "V2_LED:1608_Orange")
 		(at 129.54 57.15 0)
 		(mirror y)
@@
 	)
 	(symbol
-		(lib_id "V2_Capacitor:0805_10u")
+		(lib_id "V2_Capacitor:2012_10u")
 		(at 176.53 43.18 0)
 		(unit 1)
@@
 			)
 		)
-		(property "Footprint" "V2_Capacitor_SMD:C_0805"
+		(property "Footprint" "V2_Capacitor_SMD:C_2012"
 			(at 176.53 60.198 0)
 			(hide yes)
@@
 	)
 	(symbol
-		(lib_id "V2_Capacitor:0603_18p")
+		(lib_id "V2_Capacitor:1608_18p")
 		(at 36.83 48.26 0)
 		(unit 1)
@@
 			)
 		)
-		(property "Footprint" "V2_Capacitor_SMD:C_0603"
+		(property "Footprint" "V2_Capacitor_SMD:C_1608"
 			(at 36.83 65.278 0)
 			(hide yes)
@@
 	)
 	(symbol
-		(lib_id "V2_Capacitor:0603_10u")
+		(lib_id "V2_Capacitor:1608_10u")
 		(at 64.77 25.4 0)
 		(unit 1)
@@
 			)
 		)
-		(property "Footprint" "V2_Capacitor_SMD:C_0603"
+		(property "Footprint" "V2_Capacitor_SMD:C_1608"
 			(at 64.77 42.418 0)
 			(hide yes)
@@
 	)
 	(symbol
-		(lib_id "V2_Capacitor:0603_18p")
+		(lib_id "V2_Capacitor:1608_18p")
 		(at 31.75 48.26 0)
 		(unit 1)
@@
 			)
 		)
-		(property "Footprint" "V2_Capacitor_SMD:C_0603"
+		(property "Footprint" "V2_Capacitor_SMD:C_1608"
 			(at 31.75 65.278 0)
 			(hide yes)
@@
 	)
 	(symbol
-		(lib_id "V2_Resistor:0603_330R")
+		(lib_id "V2_Resistor:1608_330R")
 		(at 138.43 57.15 90)
 		(unit 1)
@@
 			)
 		)
-		(property "Footprint" "V2_Resistor_SMD:R_0603"
+		(property "Footprint" "V2_Resistor_SMD:R_1608"
 			(at 154.178 57.15 0)
 			(hide yes)
@@
 	)
 	(symbol
-		(lib_id "V2_Capacitor:0603_0u1")
+		(lib_id "V2_Capacitor:1608_0u1")
 		(at 105.41 25.4 0)
 		(unit 1)
@@
 			)
 		)
-		(property "Footprint" "V2_Capacitor_SMD:C_0603"
+		(property "Footprint" "V2_Capacitor_SMD:C_1608"
 			(at 105.41 42.418 0)
 			(hide yes)
@@
 	)
 	(symbol
-		(lib_id "V2_Capacitor:0805_10u")
+		(lib_id "V2_Capacitor:2012_10u")
 		(at 201.93 43.18 0)
 		(unit 1)
@@
 			)
 		)
-		(property "Footprint" "V2_Capacitor_SMD:C_0805"
+		(property "Footprint" "V2_Capacitor_SMD:C_2012"
 			(at 201.93 60.198 0)
 			(hide yes)
@@
 	)
 	(symbol
-		(lib_id "V2_Capacitor:0603_0u1")
+		(lib_id "V2_Capacitor:1608_0u1")
 		(at 85.09 25.4 0)
 		(unit 1)
@@
 			)
 		)
-		(property "Footprint" "V2_Capacitor_SMD:C_0603"
+		(property "Footprint" "V2_Capacitor_SMD:C_1608"
 			(at 85.09 42.418 0)
 			(hide yes)
@@
 	)
 	(symbol
-		(lib_id "V2_Resistor:0603_5k1")
+		(lib_id "V2_Resistor:1608_5k1")
 		(at 212.09 96.52 90)
 		(unit 1)
@@
 			)
 		)
-		(property "Footprint" "V2_Resistor_SMD:R_0603"
+		(property "Footprint" "V2_Resistor_SMD:R_1608"
 			(at 227.838 96.52 0)
 			(hide yes)
@@
 	)
 	(symbol
-		(lib_id "V2_Capacitor:0603_0u1")
+		(lib_id "V2_Capacitor:1608_0u1")
 		(at 95.25 25.4 0)
 		(unit 1)
@@
 			)
 		)
-		(property "Footprint" "V2_Capacitor_SMD:C_0603"
+		(property "Footprint" "V2_Capacitor_SMD:C_1608"
 			(at 95.25 42.418 0)
 			(hide yes)
@@
 	)
 	(symbol
-		(lib_id "V2_Resistor:0603_100k")
+		(lib_id "V2_Resistor:1608_100k")
 		(at 57.15 123.19 90)
 		(unit 1)
@@
 			)
 		)
-		(property "Footprint" "V2_Resistor_SMD:R_0603"
+		(property "Footprint" "V2_Resistor_SMD:R_1608"
 			(at 72.898 123.19 0)
 			(hide yes)
