File: hardware/strip/strip.kicad_pcb (KiCad board)
At the start: 4 copper layers, 70 x 17.5 mm, 41 parts, among them J101 Cortex, J102 DX07S016JA3, J201 WAGO 2065-100, J202 WAGO 2065-100, J203 WAGO 2065-100, SW101 SKSG, SW102 SKSG, U101 ATSAMD51G, U102 TPS78433QWDRBRQ1, U201 74AHC1G125, Y101 32k768

Commit message: Update
Parts:
- moved C103 0.75 mm to (145.5, 100.5)
- moved C104 0.75 mm to (149.5, 102.5)
- moved C105 0.50 mm to (142.5, 100.5)
- moved C107 0.50 mm to (138.2, 106.0)
Routing:
- net +3V3: track 59.5 -> 57.0 mm
- net /VDDCORE: track 2.82 -> 2.02 mm
